Commit message: finished final project

File: body.urdf (robot description, URDF)
Before this commit: robot robot, 3 links, 2 joints
Links:
- added link BackerLeg, mass 1; collision box size=1 1 1; visual box size=1 1 1
- added link FronterLeg, mass 1; collision box size=1 1 1; visual box size=1 1 1
- link Torso: geometry collision box size=1 1 2; visual box size=1 1 2
Joints:
- added joint BackLeg_BackerLeg: type revolute, parent BackLeg, child BackerLeg, origin xyz=-1 0 -1 rpy=0 0 0, axis 0 1 0, limit lower=-3.14159 upper=3.14159 effort=0.0 velocity=0.0
- added joint FrontLeg_FronterLeg: type revolute, parent FrontLeg, child FronterLeg, origin xyz=1 0 -1 rpy=0 0 0, axis 0 1 0, limit lower=-3.14159 upper=3.14159 effort=0.0 velocity=0.0
- joint Torso_BackLeg: origin xyz=1 0 1 rpy=0 0 0 -> xyz=1 0 2 rpy=0 0 0
- joint Torso_FrontLeg: origin xyz=2 0 1 rpy=0 0 0 -> xyz=2 0 2 rpy=0 0 0

Commit message: finished assignment 6

File: body.urdf (robot description, URDF)
Before this commit: robot robot, 5 links, 4 joints
Links:
- link BackLeg: geometry collision box size=0.25912471423724315 0.08941710666145686 0.02683180426767795; visual box size=0.25912471423724315 0.08941710666145686 0.02683180426767795
- link BackerLeg: geometry collision box size=0.5956261346965231 0.03825923448283053 0.7157846343796489; visual box size=0.5956261346965231 0.03825923448283053 0.7157846343796489
- link FrontLeg: geometry collision box size=0.6977765191923021 0.6074354482331922 0.8223854837895713; visual box size=0.6977765191923021 0.6074354482331922 0.8223854837895713
- link FronterLeg: geometry collision box size=0.7966238022371447 0.6580283857278536 0.012504382306862238; visual box size=0.7966238022371447 0.6580283857278536 0.012504382306862238
- link Torso: geometry collision box size=0.6821429428296557 0.7202448081696134 0.6060694455813298; visual box size=0.6821429428296557 0.7202448081696134 0.6060694455813298
Joints:
- joint BackLeg_BackerLeg: origin xyz=-1 0 -1 rpy=0 0 0 -> xyz=-0.5 0 0 rpy=0 0 0
- joint FrontLeg_FronterLeg: origin xyz=1 0 -1 rpy=0 0 0 -> xyz=0.5 0 0 rpy=0 0 0
- joint Torso_BackLeg: origin xyz=1 0 2 rpy=0 0 0 -> xyz=-0.5 0 1 rpy=0 0 0
- joint Torso_FrontLeg: origin xyz=2 0 2 rpy=0 0 0 -> xyz=0.5 0 1 rpy=0 0 0

Commit message: finished assignment 8

File: body.urdf (robot description, URDF)
Before this commit: robot robot, 5 links, 4 joints
Links:
- removed link BackLeg
- removed link BackerLeg
- removed link FrontLeg
- removed link FronterLeg
- removed link Torso
- added link Limb1, mass 1; collision box size=0.8103497743407617 0.4759950684798727 0.6209383239929874; visual box size=0.8103497743407617 0.4759950684798727 0.6209383239929874
- added link Limb2, mass 1; collision box size=0.6704172976119466 0.8158209808326184 0.7929519839530162; visual box size=0.6704172976119466 0.8158209808326184 0.7929519839530162
- added link Limb3, mass 1; collision box size=0.5384064842748424 0.971131818468372 0.9489619868403418; visual box size=0.5384064842748424 0.971131818468372 0.9489619868403418
- added link Limb4, mass 1; collision box size=0.9040909803145797 0.46739601982057244 0.4308369312876832; visual box size=0.9040909803145797 0.46739601982057244 0.4308369312876832
- added link Main, mass 1; collision box size=1.4667240303776818 1.9134301942786243 0.1334506686617907; visual box size=1.4667240303776818 1.9134301942786243 0.1334506686617907
Joints:
- removed joint BackLeg_BackerLeg
- removed joint FrontLeg_FronterLeg
- removed joint Torso_BackLeg
- removed joint Torso_FrontLeg
- added joint Main_Limb1: type revolute, parent Main, child Limb1, origin xyz=0.7333620151888409 0.6378100647595414 2.9332746656691047 rpy=0 0 0, axis 0 1 0, limit lower=-3.14159 upper=3.14159 effort=0.0 velocity=0.0
- added joint Main_Limb2: type revolute, parent Main, child Limb2, origin xyz=0.7333620151888409 -0.6378100647595414 2.9332746656691047 rpy=0 0 0, axis 0 1 0, limit lower=-3.14159 upper=3.14159 effort=0.0 velocity=0.0
- added joint Main_Limb3: type revolute, parent Main, child Limb3, origin xyz=-0.7333620151888409 0.6378100647595414 2.9332746656691047 rpy=0 0 0, axis 0 1 0, limit lower=-3.14159 upper=3.14159 effort=0.0 velocity=0.0
- added joint Main_Limb4: type revolute, parent Main, child Limb4, origin xyz=-0.7333620151888409 -0.6378100647595414 2.9332746656691047 rpy=0 0 0, axis 0 1 0, limit lower=-3.14159 upper=3.14159 effort=0.0 velocity=0.0

Commit message: finished assignment 7

File: body.urdf (robot description, URDF)
Before this commit: robot robot, 5 links, 4 joints
Links:
- link Limb1: geometry collision box size=0.12921605106727752 0.4718218055582394 0.536170700915503; visual box size=0.12921605106727752 0.4718218055582394 0.536170700915503
- link Limb2: geometry collision box size=0.02451129540508057 0.06186293439158508 0.9496577503311376; visual box size=0.02451129540508057 0.06186293439158508 0.9496577503311376
- link Limb3: geometry collision box size=0.546914716733042 0.8946989172932708 0.8071302413144522; visual box size=0.546914716733042 0.8946989172932708 0.8071302413144522
- link Limb4: geometry collision box size=0.5529632330620547 0.26761058107505276 0.4263758796529198; visual box size=0.5529632330620547 0.26761058107505276 0.4263758796529198
- link Main: geometry collision box size=0.9564503022553775 1.5307886596461462 0.3523142851462786; visual box size=0.9564503022553775 1.5307886596461462 0.3523142851462786
Joints:
- joint Main_Limb1: origin xyz=0.7333620151888409 0.6378100647595414 2.9332746656691047 rpy=0 0 0 -> xyz=0.47822515112768876 0.5102628865487154 2.8238428574268606 rpy=0 0 0
- joint Main_Limb2: origin xyz=0.7333620151888409 -0.6378100647595414 2.9332746656691047 rpy=0 0 0 -> xyz=0.47822515112768876 -0.5102628865487154 2.8238428574268606 rpy=0 0 0
- joint Main_Limb3: origin xyz=-0.7333620151888409 0.6378100647595414 2.9332746656691047 rpy=0 0 0 -> xyz=-0.47822515112768876 0.5102628865487154 2.8238428574268606 rpy=0 0 0
- joint Main_Limb4: origin xyz=-0.7333620151888409 -0.6378100647595414 2.9332746656691047 rpy=0 0 0 -> xyz=-0.47822515112768876 -0.5102628865487154 2.8238428574268606 rpy=0 0 0

Commit message: added diagram

File: body.urdf (robot description, URDF)
Before this commit: robot robot, 5 links, 4 joints
Links:
- link Limb1: geometry collision box size=0.41616600459879505 0.8962311828865054 0.08943196805974252; visual box size=0.41616600459879505 0.8962311828865054 0.08943196805974252
- link Limb2: geometry collision box size=0.9508330562338909 0.06433225698329781 0.22340108546595916; visual box size=0.9508330562338909 0.06433225698329781 0.22340108546595916
- link Limb3: geometry collision box size=0.7974969583138802 0.43469069860266685 0.9169234930322262; visual box size=0.7974969583138802 0.43469069860266685 0.9169234930322262
- link Limb4: geometry collision box size=0.7303222434890423 0.6910552066916288 0.65175820882104; visual box size=0.7303222434890423 0.6910552066916288 0.65175820882104
- link Main: geometry collision box size=0.9315962494099493 1.6564405369685749 0.7190312283398917; visual box size=0.9315962494099493 1.6564405369685749 0.7190312283398917
Joints:
- joint Main_Limb1: origin xyz=0.47822515112768876 0.5102628865487154 2.8238428574268606 rpy=0 0 0 -> xyz=0.46579812470497467 0.5521468456561917 2.640484385830054 rpy=0 0 0
- joint Main_Limb2: origin xyz=0.47822515112768876 -0.5102628865487154 2.8238428574268606 rpy=0 0 0 -> xyz=0.46579812470497467 -0.5521468456561917 2.640484385830054 rpy=0 0 0
- joint Main_Limb3: origin xyz=-0.47822515112768876 0.5102628865487154 2.8238428574268606 rpy=0 0 0 -> xyz=-0.46579812470497467 0.5521468456561917 2.640484385830054 rpy=0 0 0
- joint Main_Limb4: origin xyz=-0.47822515112768876 -0.5102628865487154 2.8238428574268606 rpy=0 0 0 -> xyz=-0.46579812470497467 -0.5521468456561917 2.640484385830054 rpy=0 0 0

Commit message: finished assignment 8

File: body.urdf (robot description, URDF)
Before this commit: robot robot, 5 links, 4 joints
Links:
- added link Limb5, mass 1; collision box size=0.3261978012429316 0.36544308087020344 0.8369201439547593; visual box size=0.3261978012429316 0.36544308087020344 0.8369201439547593
- added link Limb6, mass 1; collision box size=0.3017430673380525 0.7586155466849034 0.729605036259655; visual box size=0.3017430673380525 0.7586155466849034 0.729605036259655
- added link Limb7, mass 1; collision box size=0.6861788430991637 0.7981225715064084 0.8869301049047258; visual box size=0.6861788430991637 0.7981225715064084 0.8869301049047258
- added link Limb8, mass 1; collision box size=0.8939722247189945 0.8670925568244479 0.692413553866307; visual box size=0.8939722247189945 0.8670925568244479 0.692413553866307
- added link Limb9, mass 1; collision box size=0.6616372610114168 0.8652373564472862 0.7121301968972487; visual box size=0.6616372610114168 0.8652373564472862 0.7121301968972487
- link Limb1: geometry collision box size=0.679083644674209 0.8979175374973516 0.7201506408379509; visual box size=0.679083644674209 0.8979175374973516 0.7201506408379509
- link Limb2: geometry collision box size=0.8443561817665082 0.6962513610148271 0.650190756947826; visual box size=0.8443561817665082 0.6962513610148271 0.650190756947826
- link Limb3: geometry collision box size=0.4886230394413567 0.5622288298261 0.3996625311179157; visual box size=0.4886230394413567 0.5622288298261 0.3996625311179157
- link Limb4: geometry collision box size=0.3742490817847918 0.8437667147312529 0.3627243585312449; visual box size=0.3742490817847918 0.8437667147312529 0.3627243585312449
- link Main: geometry collision box size=0.8603136232969488 1.626408879685263 0.5325200576405197; visual box size=0.8603136232969488 1.626408879685263 0.5325200576405197
Joints:
- added joint Main_Limb5: type revolute, parent Main, child Limb5, origin xyz=-0.4301568116484744 0 3.26626002882026 rpy=0 0 0, axis 0 1 0, limit lower=-3.14159 upper=3.14159 effort=0.0 velocity=0.0
- added joint Main_Limb6: type revolute, parent Main, child Limb6, origin xyz=0.4301568116484744 0 3.26626002882026 rpy=0 0 0, axis 0 1 0, limit lower=-3.14159 upper=3.14159 effort=0.0 velocity=0.0
- added joint Main_Limb7: type revolute, parent Main, child Limb7, origin xyz=0 0 3.26626002882026 rpy=0 0 0, axis 0 1 0, limit lower=-3.14159 upper=3.14159 effort=0.0 velocity=0.0
- added joint Main_Limb8: type revolute, parent Main, child Limb8, origin xyz=0 -0.8132044398426315 3 rpy=0 0 0, axis 0 1 0, limit lower=-3.14159 upper=3.14159 effort=0.0 velocity=0.0
- added joint Main_Limb9: type revolute, parent Main, child Limb9, origin xyz=0 0.8132044398426315 3 rpy=0 0 0, axis 0 1 0, limit lower=-3.14159 upper=3.14159 effort=0.0 velocity=0.0
- joint Main_Limb1: origin xyz=0.46579812470497467 0.5521468456561917 2.640484385830054 rpy=0 0 0 -> xyz=0.4301568116484744 0.5421362932284209 2.73373997117974 rpy=0 0 0
- joint Main_Limb2: origin xyz=0.46579812470497467 -0.5521468456561917 2.640484385830054 rpy=0 0 0 -> xyz=0.4301568116484744 -0.5421362932284209 2.73373997117974 rpy=0 0 0
- joint Main_Limb3: origin xyz=-0.46579812470497467 0.5521468456561917 2.640484385830054 rpy=0 0 0 -> xyz=-0.4301568116484744 0.5421362932284209 2.73373997117974 rpy=0 0 0
- joint Main_Limb4: origin xyz=-0.46579812470497467 -0.5521468456561917 2.640484385830054 rpy=0 0 0 -> xyz=-0.4301568116484744 -0.5421362932284209 2.73373997117974 rpy=0 0 0
